File: output/pcbs/main.kicad_pcb (KiCad board)
At the start: 2 copper layers, 251.9 x 126.1 mm, 145 parts

Commit message: Also commit this too
Parts:
- removed ?: , ProMicro
- removed S100, S103, S106, S73, S76, S79, S82, S85, S88, S91, S94, S97: , MX
- removed S101, S104, S107, S74, S77, S80, S83, S86, S89, S92, S95, S98: , ALPS
- removed S102, S105, S108, S75, S78, S81, S84, S87, S90, S93, S96, S99: , PG1350
- added MCU1: , ProMicro, F.Cu at (109.3, 14.2)
- S10, S16, S22, S28, S34, S4, S40, S46, S52, S58, S64, S70: footprint MX -> PG1350
- S11, S17, S23, S29, S35, S41, S47, S5, S53, S59, S65, S71: footprint ALPS -> MX
- S14, S2, S20, S26, S32, S38, S44, S50, S56, S62, S68, S8: footprint ALPS -> PG1350
- S15, S21, S27, S3, S33, S39, S45, S51, S57, S63, S69, S9: footprint PG1350 -> MX
- moved S37 153.4 mm to (225.7, -29.8), turned to 25 degrees
- moved S38 153.4 mm to (225.7, -29.8), turned to 25 degrees
- moved S39 135.6 mm to (210.6, -17.2), turned to 25 degrees
- moved S47 130.2 mm to (176.0, -46.3), turned to 25 degrees
- moved S48 130.2 mm to (176.0, -46.3), turned to 25 degrees
- moved S46 128.1 mm to (184.1, -29.1), turned to 25 degrees
- moved S40 125.0 mm to (210.6, -17.2), turned to 25 degrees
- moved S53 123.1 mm to (155.9, -44.7), turned to 25 degrees
- moved S54 123.1 mm to (155.9, -44.7), turned to 25 degrees
- moved S41 120.0 mm to (202.6, -34.4), turned to 25 degrees
- moved S42 120.0 mm to (202.6, -34.4), turned to 25 degrees
- moved S71 117.8 mm to (126.6, 60.6)
- moved S72 117.8 mm to (126.6, 60.6)
- moved S52 113.6 mm to (163.9, -27.4), turned to 25 degrees
- moved S51 100.3 mm to (163.9, -27.4), turned to 25 degrees
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Connections:
- D1 pad 1: pinky_bottom -> !colrow
- D1 pad 2: P16 -> !row_net
- D10 pad 1: index_bottom -> !colrow
- D10 pad 2: P16 -> !row_net
- D11 pad 1: index_home -> !colrow
- D11 pad 2: P15 -> !row_net
- D12 pad 1: index_top -> !colrow
- D12 pad 2: P20 -> !row_net
- D13 pad 1: inner_bottom -> !colrow
- D13 pad 2: P16 -> !row_net
- D14 pad 1: inner_home -> !colrow
- D14 pad 2: P15 -> !row_net
- D15 pad 1: inner_top -> !colrow
- D15 pad 2: P20 -> !row_net
- D16 pad 1: near_thumb -> !colrow
- D16 pad 2: P10 -> !row_net
- D17 pad 1: home_thumb -> !colrow
- D17 pad 2: P10 -> !row_net
- D18 pad 1: far_thumb -> !colrow
- D18 pad 2: P10 -> !row_net
- D19 pad 1: mirror_pinky_bottom -> !colrow
- D19 pad 2: P9 -> !row_net
- D2 pad 1: pinky_home -> !colrow
- D2 pad 2: P15 -> !row_net
- D20 pad 1: mirror_pinky_home -> !colrow
- D20 pad 2: P6 -> !row_net
- D21 pad 1: mirror_pinky_top -> !colrow
- D21 pad 2: P2 -> !row_net
- D22 pad 1: mirror_ring_bottom -> !colrow
- D22 pad 2: P9 -> !row_net
- D23 pad 1: mirror_ring_home -> !colrow
- D23 pad 2: P6 -> !row_net
- D24 pad 1: mirror_ring_top -> !colrow
- D24 pad 2: P2 -> !row_net
- D25 pad 1: mirror_middle_bottom -> !colrow
- D25 pad 2: P9 -> !row_net
- D26 pad 1: mirror_middle_home -> !colrow
- D26 pad 2: P6 -> !row_net
- D27 pad 1: mirror_middle_top -> !colrow
- D27 pad 2: P2 -> !row_net
- D28 pad 1: mirror_index_bottom -> !colrow
- D28 pad 2: P9 -> !row_net
- D29 pad 1: mirror_index_home -> !colrow
- D29 pad 2: P6 -> !row_net
- D3 pad 1: pinky_top -> !colrow
- D3 pad 2: P20 -> !row_net
- D30 pad 1: mirror_index_top -> !colrow
- D30 pad 2: P2 -> !row_net
- D31 pad 1: mirror_inner_bottom -> !colrow
- D31 pad 2: P9 -> !row_net
- D32 pad 1: mirror_inner_home -> !colrow
- D32 pad 2: P6 -> !row_net
- D33 pad 1: mirror_inner_top -> !colrow
- D33 pad 2: P2 -> !row_net
- D34 pad 1: mirror_near_thumb -> !colrow
- D34 pad 2: P19 -> !row_net
- D35 pad 1: mirror_home_thumb -> !colrow
- D35 pad 2: P19 -> !row_net
- D36 pad 1: mirror_far_thumb -> !colrow
- D36 pad 2: P19 -> !row_net
- D4 pad 1: ring_bottom -> !colrow
- D4 pad 2: P16 -> !row_net
- D5 pad 1: ring_home -> !colrow
- D5 pad 2: P15 -> !row_net
- D6 pad 1: ring_top -> !colrow
- D6 pad 2: P20 -> !row_net
- D7 pad 1: middle_bottom -> !colrow
- D7 pad 2: P16 -> !row_net
- D8 pad 1: middle_home -> !colrow
- D8 pad 2: P15 -> !row_net
- D9 pad 1: middle_top -> !colrow
- D9 pad 2: P20 -> !row_net
- S1 pad 1: pinky_bottom -> !colrow
- S1 pad 2: P4 -> !column_net
- S10 pad 1: ring_bottom -> !colrow
- S10 pad 2: P5 -> !column_net
- S11 pad 1: ring_bottom -> !colrow
- S11 pad 2: P5 -> !column_net
- S12 pad 1: ring_bottom -> !colrow
- S12 pad 2: P5 -> !column_net
- S13 pad 1: ring_home -> !colrow
- S13 pad 2: P5 -> !column_net
- S14 pad 1: ring_home -> !colrow
- S14 pad 2: P5 -> !column_net
- S15 pad 1: ring_home -> !colrow
- S15 pad 2: P5 -> !column_net
- S16 pad 1: ring_top -> !colrow
- S16 pad 2: P5 -> !column_net
- S17 pad 1: ring_top -> !colrow
- S17 pad 2: P5 -> !column_net
- S18 pad 1: ring_top -> !colrow
- S18 pad 2: P5 -> !column_net
- S19 pad 1: middle_bottom -> !colrow
- S19 pad 2: P7 -> !column_net
- S2 pad 1: pinky_bottom -> !colrow
- S2 pad 2: P4 -> !column_net
- S20 pad 1: middle_bottom -> !colrow
- S20 pad 2: P7 -> !column_net
- S21 pad 1: middle_bottom -> !colrow
- S21 pad 2: P7 -> !column_net
- S22 pad 1: middle_home -> !colrow
- S22 pad 2: P7 -> !column_net
- S23 pad 1: middle_home -> !colrow
- S23 pad 2: P7 -> !column_net
- S24 pad 1: middle_home -> !colrow
- S24 pad 2: P7 -> !column_net
- S25 pad 1: middle_top -> !colrow
- S25 pad 2: P7 -> !column_net
- S26 pad 1: middle_top -> !colrow
- S26 pad 2: P7 -> !column_net
- S27 pad 1: middle_top -> !colrow
- S27 pad 2: P7 -> !column_net
- S28 pad 1: index_bottom -> !colrow
- S28 pad 2: P8 -> !column_net
- S29 pad 1: index_bottom -> !colrow
- S29 pad 2: P8 -> !column_net
- S3 pad 1: pinky_bottom -> !colrow
- S3 pad 2: P4 -> !column_net
- S30 pad 1: index_bottom -> !colrow
- S30 pad 2: P8 -> !column_net
- S31 pad 1: index_home -> !colrow
- S31 pad 2: P8 -> !column_net
- S32 pad 1: index_home -> !colrow
- S32 pad 2: P8 -> !column_net
- S33 pad 1: index_home -> !colrow
- S33 pad 2: P8 -> !column_net
- S34 pad 1: index_top -> !colrow
- S34 pad 2: P8 -> !column_net
- S35 pad 1: index_top -> !colrow
- S35 pad 2: P8 -> !column_net
- S36 pad 1: index_top -> !colrow
- S36 pad 2: P8 -> !column_net
- S37 pad 1: inner_bottom -> !column_net
- S37 pad 2: P1 -> !colrow
- S38 pad 1: inner_bottom -> !column_net
- S38 pad 2: P1 -> !colrow
- S39 pad 1: inner_bottom -> !column_net
- S39 pad 2: P1 -> !colrow
- S4 pad 1: pinky_home -> !colrow
- S4 pad 2: P4 -> !column_net
- S40 pad 1: inner_home -> !column_net
- S40 pad 2: P1 -> !colrow
- S41 pad 1: inner_home -> !column_net
- S41 pad 2: P1 -> !colrow
- S42 pad 1: inner_home -> !column_net
- S42 pad 2: P1 -> !colrow
- S43 pad 1: inner_top -> !column_net
- S43 pad 2: P1 -> !colrow
- S44 pad 1: inner_top -> !column_net
- S44 pad 2: P1 -> !colrow
- S45 pad 1: inner_top -> !column_net
- S45 pad 2: P1 -> !colrow
- S46 pad 1: near_thumb -> !column_net
- S46 pad 2: P7 -> !colrow
- S47 pad 1: near_thumb -> !column_net
- S47 pad 2: P7 -> !colrow
- S48 pad 1: near_thumb -> !column_net
- S48 pad 2: P7 -> !colrow
- S49 pad 1: home_thumb -> !column_net
- S49 pad 2: P8 -> !colrow
- S5 pad 1: pinky_home -> !colrow
- S5 pad 2: P4 -> !column_net
- S50 pad 1: home_thumb -> !column_net
- S50 pad 2: P8 -> !colrow
- S51 pad 1: home_thumb -> !column_net
- S51 pad 2: P8 -> !colrow
- S52 pad 1: far_thumb -> !column_net
- S52 pad 2: P1 -> !colrow
- S53 pad 1: far_thumb -> !column_net
- S53 pad 2: P1 -> !colrow
- S54 pad 1: far_thumb -> !column_net
- S54 pad 2: P1 -> !colrow
- S55 pad 1: P4 -> !column_net
- S55 pad 2: mirror_pinky_bottom -> !colrow
- S56 pad 1: P4 -> !column_net
- S56 pad 2: mirror_pinky_bottom -> !colrow
- S57 pad 1: P4 -> !column_net
- S57 pad 2: mirror_pinky_bottom -> !colrow
- S58 pad 1: P4 -> !column_net
- S58 pad 2: mirror_pinky_home -> !colrow
- S59 pad 1: P4 -> !column_net
- S59 pad 2: mirror_pinky_home -> !colrow
- S6 pad 1: pinky_home -> !colrow
- S6 pad 2: P4 -> !column_net
- S60 pad 1: P4 -> !column_net
- S60 pad 2: mirror_pinky_home -> !colrow
- S61 pad 1: P4 -> !column_net
- S61 pad 2: mirror_pinky_top -> !colrow
- S62 pad 1: P4 -> !column_net
- S62 pad 2: mirror_pinky_top -> !colrow
- S63 pad 1: P4 -> !column_net
- S63 pad 2: mirror_pinky_top -> !colrow
- S64 pad 1: P5 -> !column_net
- S64 pad 2: mirror_ring_bottom -> !colrow
- S65 pad 1: P5 -> !column_net
- S65 pad 2: mirror_ring_bottom -> !colrow
- S66 pad 1: P5 -> !column_net
- S66 pad 2: mirror_ring_bottom -> !colrow
- S67 pad 1: P5 -> !colrow
- S67 pad 2: mirror_ring_home -> !column_net
- S68 pad 1: P5 -> !colrow
- S68 pad 2: mirror_ring_home -> !column_net
- S69 pad 1: P5 -> !colrow
- S69 pad 2: mirror_ring_home -> !column_net
- S7 pad 1: pinky_top -> !colrow
- S7 pad 2: P4 -> !column_net
- S70 pad 1: P5 -> !colrow
- S70 pad 2: mirror_ring_top -> !column_net
- S71 pad 1: P5 -> !colrow
- S71 pad 2: mirror_ring_top -> !column_net
- S72 pad 1: P5 -> !colrow
- S72 pad 2: mirror_ring_top -> !column_net
- S8 pad 1: pinky_top -> !colrow
- S8 pad 2: P4 -> !column_net
- S9 pad 1: pinky_top -> !colrow
- S9 pad 2: P4 -> !column_net
Other:
- outline, holes or cut-outs redrawn

Commit message: Routing fixed, added encoder and on / off switch.  Last that is left is JST connector and reset button
Parts:
- added OLED1: OLED, lib:OLED_headers, F.Cu at (103.6, 32.2)
- added ROT1: , rotary_encoder, F.Cu at (109.3, 41.2)
- added T1: , E73:SPDT_C128955, F.Cu at (109.3, 51.2)
Connections:
- D1 pad 1: !colrow -> pinky_bottom
- D1 pad 2: !row_net -> P18
- D10 pad 1: !colrow -> index_bottom
- D10 pad 2: !row_net -> P18
- D11 pad 1: !colrow -> index_home
- D11 pad 2: !row_net -> P19
- D12 pad 1: !colrow -> index_top
- D12 pad 2: !row_net -> P20
- D13 pad 1: !colrow -> inner_bottom
- D13 pad 2: !row_net -> P18
- D14 pad 1: !colrow -> inner_home
- D14 pad 2: !row_net -> P19
- D15 pad 1: !colrow -> inner_top
- D15 pad 2: !row_net -> P20
- D16 pad 1: !colrow -> near_thumb
- D16 pad 2: !row_net -> P20
- D17 pad 1: !colrow -> home_thumb
- D17 pad 2: !row_net -> P19
- D18 pad 1: !colrow -> far_thumb
- D18 pad 2: !row_net -> P18
- D19 pad 1: !colrow -> mirror_pinky_bottom
- D19 pad 2: !row_net -> P4
- D2 pad 1: !colrow -> pinky_home
- D2 pad 2: !row_net -> P19
- D20 pad 1: !colrow -> mirror_pinky_home
- D20 pad 2: !row_net -> P5
- D21 pad 1: !colrow -> mirror_pinky_top
- D21 pad 2: !row_net -> P6
- D22 pad 1: !colrow -> mirror_ring_bottom
- D22 pad 2: !row_net -> P4
- D23 pad 1: !colrow -> mirror_ring_home
- D23 pad 2: !row_net -> P5
- D24 pad 1: !colrow -> mirror_ring_top
- D24 pad 2: !row_net -> P6
- D25 pad 1: !colrow -> mirror_middle_bottom
- D25 pad 2: !row_net -> P4
- D26 pad 1: !colrow -> mirror_middle_home
- D26 pad 2: !row_net -> P5
- D27 pad 1: !colrow -> mirror_middle_top
- D27 pad 2: !row_net -> P6
- D28 pad 1: !colrow -> mirror_index_bottom
- D28 pad 2: !row_net -> P4
- D29 pad 1: !colrow -> mirror_index_home
- D29 pad 2: !row_net -> P5
- D3 pad 1: !colrow -> pinky_top
- D3 pad 2: !row_net -> P20
- D30 pad 1: !colrow -> mirror_index_top
- D30 pad 2: !row_net -> P6
- D31 pad 1: !colrow -> mirror_inner_bottom
- D31 pad 2: !row_net -> P4
- D32 pad 1: !colrow -> mirror_inner_home
- D32 pad 2: !row_net -> P5
- D33 pad 1: !colrow -> mirror_inner_top
- D33 pad 2: !row_net -> P6
- D34 pad 1: !colrow -> mirror_near_thumb
- D34 pad 2: !row_net -> P6
- D35 pad 1: !colrow -> mirror_home_thumb
- D35 pad 2: !row_net -> P5
- D36 pad 1: !colrow -> mirror_far_thumb
- D36 pad 2: !row_net -> P4
- D4 pad 1: !colrow -> ring_bottom
- D4 pad 2: !row_net -> P18
- D5 pad 1: !colrow -> ring_home
- D5 pad 2: !row_net -> P19
- D6 pad 1: !colrow -> ring_top
- D6 pad 2: !row_net -> P20
- D7 pad 1: !colrow -> middle_bottom
- D7 pad 2: !row_net -> P18
- D8 pad 1: !colrow -> middle_home
- D8 pad 2: !row_net -> P19
- D9 pad 1: !colrow -> middle_top
- D9 pad 2: !row_net -> P20
- S1 pad 1: !colrow -> pinky_bottom
- S1 pad 2: !column_net -> P9
- S10 pad 1: !colrow -> ring_home
- S10 pad 2: !column_net -> P10
- S11 pad 1: !colrow -> ring_top
- S11 pad 2: !column_net -> P10
- S12 pad 1: !colrow -> ring_top
- S12 pad 2: !column_net -> P10
- S13 pad 1: !colrow -> middle_bottom
- S13 pad 2: !column_net -> P8
- S14 pad 1: !colrow -> middle_bottom
- S14 pad 2: !column_net -> P8
- S15 pad 1: !colrow -> middle_home
- S15 pad 2: !column_net -> P8
- S16 pad 1: !colrow -> middle_home
- S16 pad 2: !column_net -> P8
- S17 pad 1: !colrow -> middle_top
- S17 pad 2: !column_net -> P8
- S18 pad 1: !colrow -> middle_top
- S18 pad 2: !column_net -> P8
- S19 pad 1: !colrow -> index_bottom
- S19 pad 2: !column_net -> P16
- S2 pad 1: !colrow -> pinky_bottom
- S2 pad 2: !column_net -> P9
- S20 pad 1: !colrow -> index_bottom
- S20 pad 2: !column_net -> P16
- S21 pad 1: !colrow -> index_home
- S21 pad 2: !column_net -> P16
- S22 pad 1: !colrow -> index_home
- S22 pad 2: !column_net -> P16
- S23 pad 1: !colrow -> index_top
- S23 pad 2: !column_net -> P16
- S24 pad 1: !colrow -> index_top
- S24 pad 2: !column_net -> P16
- S25 pad 1: !colrow -> inner_bottom
- S25 pad 2: !column_net -> P7
- S26 pad 1: !colrow -> inner_bottom
- S26 pad 2: !column_net -> P7
- S27 pad 1: !colrow -> inner_home
- S27 pad 2: !column_net -> P7
- S28 pad 1: !colrow -> inner_home
- S28 pad 2: !column_net -> P7
- S29 pad 1: !colrow -> inner_top
- S29 pad 2: !column_net -> P7
- S3 pad 1: !colrow -> pinky_home
- S3 pad 2: !column_net -> P9
- S30 pad 1: !colrow -> inner_top
- S30 pad 2: !column_net -> P7
- S31 pad 1: !colrow -> near_thumb
- S31 pad 2: !column_net -> P14
- S32 pad 1: !colrow -> near_thumb
- S32 pad 2: !column_net -> P14
- S33 pad 1: !colrow -> home_thumb
- S33 pad 2: !column_net -> P14
- S34 pad 1: !colrow -> home_thumb
- S34 pad 2: !column_net -> P14
- S35 pad 1: !colrow -> far_thumb
- S35 pad 2: !column_net -> P14
- S36 pad 1: !colrow -> far_thumb
- S36 pad 2: !column_net -> P14
- S37 pad 1: !column_net -> P9
- S37 pad 2: !colrow -> mirror_pinky_bottom
- S38 pad 1: !column_net -> P9
- S38 pad 2: !colrow -> mirror_pinky_bottom
- S39 pad 1: !column_net -> P9
- S39 pad 2: !colrow -> mirror_pinky_home
- S4 pad 1: !colrow -> pinky_home
- S4 pad 2: !column_net -> P9
- S40 pad 1: !column_net -> P9
- S40 pad 2: !colrow -> mirror_pinky_home
- S41 pad 1: !column_net -> P9
- S41 pad 2: !colrow -> mirror_pinky_top
- S42 pad 1: !column_net -> P9
- S42 pad 2: !colrow -> mirror_pinky_top
- S43 pad 1: !column_net -> P10
- S43 pad 2: !colrow -> mirror_ring_bottom
- S44 pad 1: !column_net -> P10
- S44 pad 2: !colrow -> mirror_ring_bottom
- S45 pad 1: !column_net -> P10
- S45 pad 2: !colrow -> mirror_ring_home
- S46 pad 1: !column_net -> P10
- S46 pad 2: !colrow -> mirror_ring_home
- S47 pad 1: !column_net -> P10
- S47 pad 2: !colrow -> mirror_ring_top
- S48 pad 1: !column_net -> P10
- S48 pad 2: !colrow -> mirror_ring_top
- S49 pad 1: !column_net -> P8
- S49 pad 2: !colrow -> mirror_middle_bottom
- S5 pad 1: !colrow -> pinky_top
- S5 pad 2: !column_net -> P9
- S50 pad 1: !column_net -> P8
- S50 pad 2: !colrow -> mirror_middle_bottom
- S51 pad 1: !column_net -> P8
- S51 pad 2: !colrow -> mirror_middle_home
- S52 pad 1: !column_net -> P8
- S52 pad 2: !colrow -> mirror_middle_home
- S53 pad 1: !column_net -> P8
- S53 pad 2: !colrow -> mirror_middle_top
- S54 pad 1: !column_net -> P8
- S54 pad 2: !colrow -> mirror_middle_top
- S55 pad 1: !column_net -> P16
- S55 pad 2: !colrow -> mirror_index_bottom
- S56 pad 1: !column_net -> P16
- S56 pad 2: !colrow -> mirror_index_bottom
- S57 pad 1: !column_net -> P16
- S57 pad 2: !colrow -> mirror_index_home
- S58 pad 1: !column_net -> P16
- S58 pad 2: !colrow -> mirror_index_home
- S59 pad 1: !column_net -> P16
- S59 pad 2: !colrow -> mirror_index_top
- S6 pad 1: !colrow -> pinky_top
- S6 pad 2: !column_net -> P9
- S60 pad 1: !column_net -> P16
- S60 pad 2: !colrow -> mirror_index_top
- S61 pad 1: !column_net -> P7
- S61 pad 2: !colrow -> mirror_inner_bottom
- S62 pad 1: !column_net -> P7
- S62 pad 2: !colrow -> mirror_inner_bottom
- S63 pad 1: !column_net -> P7
- S63 pad 2: !colrow -> mirror_inner_home
- S64 pad 1: !column_net -> P7
- S64 pad 2: !colrow -> mirror_inner_home
- S65 pad 1: !column_net -> P7
- S65 pad 2: !colrow -> mirror_inner_top
- S66 pad 1: !column_net -> P7
- S66 pad 2: !colrow -> mirror_inner_top
- S67 pad 1: !colrow -> mirror_near_thumb
- S67 pad 2: !column_net -> P14
- S68 pad 1: !colrow -> mirror_near_thumb
- S68 pad 2: !column_net -> P14
- S69 pad 1: !colrow -> mirror_home_thumb
- S69 pad 2: !column_net -> P14
- S7 pad 1: !colrow -> ring_bottom
- S7 pad 2: !column_net -> P10
- S70 pad 1: !colrow -> mirror_home_thumb
- S70 pad 2: !column_net -> P14
- S71 pad 1: !colrow -> mirror_far_thumb
- S71 pad 2: !column_net -> P14
- S72 pad 1: !colrow -> mirror_far_thumb
- S72 pad 2: !column_net -> P14
- S8 pad 1: !colrow -> ring_bottom
- S8 pad 2: !column_net -> P10
- S9 pad 1: !colrow -> ring_home
- S9 pad 2: !column_net -> P10

Commit message: Added reset button
Parts:
- added B1: , E73:SW_TACT_ALPS_SKQGABE010, F.Cu at (94.3, 12.2)
- added JST1: , JST_PH_S2B-PH-K_02x2.00mm_Angled, F.Cu at (107.3, 35.7)
- moved T1 53.0 mm to (109.3, -1.82), turned to 0 degrees
- moved ROT1 4.50 mm to (109.3, 45.7)
- moved OLED1 0.50 mm to (103.6, 32.7)
Changed lines of the file:
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@@
       )
         (module lib:OLED_headers (layer F.Cu)
-          (at 103.5547551 32.1802166 90)
+          (at 103.5547551 32.6802166 90)
           (fp_text
             reference "OLED1"
@@
         )
         (module rotary_encoder (layer F.Cu)
-            (at 109.3047551 41.1802166 0)
+            (at 109.3047551 45.6802166 0)
             (fp_text reference "ROT1" (at 0 0.5) (layer F.SilkS)
                 hide (effects (font (size 1 1) (thickness 0.15))))
@@
         )
         (module E73:SPDT_C128955 (layer F.Cu)
-            (at 109.3047551 51.1802166 180)
+            (at 109.3047551 -1.8197834000000004 0)
             (fp_text reference "T1" (at 0 0) (layer F.SilkS) hide (effects (font (size 1.27 1.27) (thickness 0.15))))
             (fp_text value "" (at 0 0) (layer F.SilkS) hide (effects (font (size 1.27 1.27) (thickness 0.15))))
@@
             (pad "" np_thru_hole circle (at 1.5 0) (size 1 1) (drill 0.9) (layers *.Cu *.Mask))
             (pad "" np_thru_hole circle (at -1.5 0) (size 1 1) (drill 0.9) (layers *.Cu *.Mask))
-            (pad 1 smd rect (at 2.25 2.075 180) (size 0.9 1.25) (layers F.Cu F.Paste F.Mask) (net 50 "GND"))
-            (pad 2 smd rect (at -0.75 2.075 180) (size 0.9 1.25) (layers F.Cu F.Paste F.Mask) (net 50 "GND"))
-            (pad 3 smd rect (at -2.25 2.075 180) (size 0.9 1.25) (layers F.Cu F.Paste F.Mask))
-            (pad "" smd rect (at 3.7 -1.1 180) (size 0.9 0.9) (layers F.Cu F.Paste F.Mask))
-            (pad "" smd rect (at 3.7 1.1 180) (size 0.9 0.9) (layers F.Cu F.Paste F.Mask))
-            (pad "" smd rect (at -3.7 1.1 180) (size 0.9 0.9) (layers F.Cu F.Paste F.Mask))
-            (pad "" smd rect (at -3.7 -1.1 180) (size 0.9 0.9) (layers F.Cu F.Paste F.Mask))
+            (pad 1 smd rect (at 2.25 2.075 0) (size 0.9 1.25) (layers F.Cu F.Paste F.Mask) (net 50 "GND"))
+            (pad 2 smd rect (at -0.75 2.075 0) (size 0.9 1.25) (layers F.Cu F.Paste F.Mask) (net 50 "GND"))
+            (pad 3 smd rect (at -2.25 2.075 0) (size 0.9 1.25) (layers F.Cu F.Paste F.Mask))
+            (pad "" smd rect (at 3.7 -1.1 0) (size 0.9 0.9) (layers F.Cu F.Paste F.Mask))
+            (pad "" smd rect (at 3.7 1.1 0) (size 0.9 0.9) (layers F.Cu F.Paste F.Mask))
+            (pad "" smd rect (at -3.7 1.1 0) (size 0.9 0.9) (layers F.Cu F.Paste F.Mask))
+            (pad "" smd rect (at -3.7 -1.1 0) (size 0.9 0.9) (layers F.Cu F.Paste F.Mask))
         )
+    (module JST_PH_S2B-PH-K_02x2.00mm_Angled (layer F.Cu)
+        (descr "JST PH series connector, S2B-PH-K, side entry type, through hole, Datasheet: http://www.jst-mfg.com/product/pdf/eng/ePH.pdf")
+        (tags "connector jst ph")
+        (at 107.3047551 35.6802166 90)
+        (fp_text reference "JST1" (at 0 0) (layer F.SilkS) hide (effects (font (size 1.27 1.27) (thickness 0.15))))
+        (fp_text value "" (at 0 0) (layer F.SilkS) hide (effects (font (size 1.27 1.27) (thickness 0.15))))
+        (fp_line (start -2.25 0.25) (end -2.25 -1.35) (layer F.SilkS) (width 0.15))
+        (fp_line (start -2.25 -1.35) (end -2.95 -1.35) (layer F.SilkS) (width 0.15))
+        (fp_line (start -2.95 -1.35) (end -2.95 6.25) (layer F.SilkS) (width 0.15))
+        (fp_line (start -2.95 6.25) (end 2.95 6.25) (layer F.SilkS) (width 0.15))
+        (fp_line (start 2.95 6.25) (end 2.95 -1.35) (layer F.SilkS) (width 0.15))
+        (fp_line (start 2.95 -1.35) (end 2.25 -1.35) (layer F.SilkS) (width 0.15))
+        (fp_line (start 2.25 -1.35) (end 2.25 0.25) (layer F.SilkS) (width 0.15))
+        (fp_line (start 2.25 0.25) (end -2.25 0.25) (layer F.SilkS) (width 0.15))
+        (fp_line (start -1 1.5) (end -1 2.0) (layer F.SilkS) (width 0.15))
+        (fp_line (start -1.25 1.75) (end -0.75 1.75) (layer F.SilkS) (width 0.15))
+        (pad 1 thru_hole rect (at -1 0 90) (size 1.2 1.7) (drill 0.75) (layers *.Cu *.Mask) (net 49 "RAW"))
+        (pad 2 thru_hole oval (at 1 0 90) (size 1.2 1.7) (drill 0.75) (layers *.Cu *.Mask) (net 50 "GND"))
+    )
+    (module E73:SW_TACT_ALPS_SKQGABE010 (layer F.Cu)
+        (descr "Low-profile SMD Tactile Switch, https://www.e-switch.com/product-catalog/tact/product-lines/tl3342-series-low-profile-smt-tact-switch")
+        (tags "SPST Tactile Switch")
+        (at 94.3047551 12.1802166 -115)
+        (fp_text reference "B1" (at 0 0) (layer F.SilkS) hide (effects (font (size 1.27 1.27) (thickness 0.15))))
+        (fp_text value "" (at 0 0) (layer F.SilkS) hide (effects (font (size 1.27 1.27) (thickness 0.15))))
+        (fp_line (start 2.75 1.25) (end 1.25 2.75) (layer F.SilkS) (width 0.15))
+        (fp_line (start 2.75 -1.25) (end 1.25 -2.75) (layer F.SilkS) (width 0.15))
+        (fp_line (start 2.75 -1.25) (end 2.75 1.25) (layer F.SilkS) (width 0.15))
+        (fp_line (start -1.25 2.75) (end 1.25 2.75) (layer F.SilkS) (width 0.15))
+        (fp_line (start -1.25 -2.75) (end 1.25 -2.75) (layer F.SilkS) (width 0.15))
+        (fp_line (start -2.75 1.25) (end -1.25 2.75) (layer F.SilkS) (width 0.15))
+        (fp_line (start -2.75 -1.25) (end -1.25 -2.75) (layer F.SilkS) (width 0.15))
+        (fp_line (start -2.75 -1.25) (end -2.75 1.25) (layer F.SilkS) (width 0.15))
+        (pad 1 smd rect (at -3.1 -1.85 -115) (size 1.8 1.1) (layers F.Cu F.Paste F.Mask) (net 51 "RST"))
+        (pad 1 smd rect (at 3.1 -1.85 -115) (size 1.8 1.1) (layers F.Cu F.Paste F.Mask) (net 51 "RST"))
+        (pad 2 smd rect (at -3.1 1.85 -115) (size 1.8 1.1) (layers F.Cu F.Paste F.Mask) (net 50 "GND"))
+        (pad 2 smd rect (at 3.1 1.85 -115) (size 1.8 1.1) (layers F.Cu F.Paste F.Mask) (net 50 "GND"))
+    )
             (gr_line (start -16.6452773 -26.2985693) (end 0.5745706930173977 -18.26882230166035) (angle 90) (layer Edge.Cuts) (width 0.15))
 (gr_line (start -10.559574300000001 -39.3494015) (end 6.660273653731254 -31.319654519979782) (angle 90) (layer Edge.Cuts) (width 0.15))

Commit message: Flipped the JST connector to be correct
Parts:
- moved D33 168.1 mm to (220.7, 118.3)
- moved S67 168.1 mm to (250.6, 162.9)
- moved S68 168.1 mm to (250.6, 162.9)
- moved S31 168.1 mm to (172.3, 162.9)
- moved S32 168.1 mm to (172.3, 162.9)
- moved S33 168.1 mm to (189.5, 170.9)
- moved S34 168.1 mm to (189.5, 170.9)
- moved S69 168.1 mm to (233.4, 170.9)
- moved S70 168.1 mm to (233.4, 170.9)
- moved S27 168.1 mm to (188.4, 128.4)
- moved S28 168.1 mm to (188.4, 128.4)
- moved D15 168.1 mm to (202.2, 118.3)
- moved S19 168.1 mm to (163.1, 137.6)
- moved S20 168.1 mm to (163.1, 137.6)
- moved S25 168.1 mm to (180.3, 145.6)
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Connections:
- D1 pad 1: pinky_bottom -> P18
- D10 pad 1: index_bottom -> P18
- D11 pad 2: P19 -> index_home
- D12 pad 1: index_top -> P20
- D12 pad 2: P20 -> index_top
- D13 pad 2: P18 -> inner_bottom
- D14 pad 2: P19 -> inner_home
- D15 pad 1: inner_top -> P20
- D15 pad 2: P20 -> inner_top
- D17 pad 1: home_thumb -> P19
- D17 pad 2: P19 -> home_thumb
- D18 pad 1: far_thumb -> P18
- D19 pad 2: P4 -> mirror_pinky_bottom
- D2 pad 2: P19 -> pinky_home
- D20 pad 1: mirror_pinky_home -> P5
- D20 pad 2: P5 -> mirror_pinky_home
- D21 pad 1: mirror_pinky_top -> P6
- D21 pad 2: P6 -> mirror_pinky_top
- D22 pad 1: mirror_ring_bottom -> P4
- D24 pad 1: mirror_ring_top -> P6
- D24 pad 2: P6 -> mirror_ring_top
- D25 pad 1: mirror_middle_bottom -> P4
- D25 pad 2: P4 -> mirror_middle_bottom
- D27 pad 1: mirror_middle_top -> P6
- D28 pad 1: mirror_index_bottom -> P4
- D29 pad 1: mirror_index_home -> P5
- D29 pad 2: P5 -> mirror_index_home
- D3 pad 1: pinky_top -> P20
- D3 pad 2: P20 -> pinky_top
- D30 pad 2: P6 -> mirror_index_top
- D31 pad 1: mirror_inner_bottom -> P4
- D32 pad 1: mirror_inner_home -> P5
- D32 pad 2: P5 -> mirror_inner_home
- D33 pad 2: P6 -> mirror_inner_top
- D34 pad 2: P6 -> mirror_near_thumb
- D35 pad 1: mirror_home_thumb -> P5
- D35 pad 2: P5 -> mirror_home_thumb
- D36 pad 1: mirror_far_thumb -> P4
- D36 pad 2: P4 -> mirror_far_thumb
- D4 pad 1: ring_bottom -> P18
- D5 pad 1: ring_home -> P19
- D5 pad 2: P19 -> ring_home
- D7 pad 1: middle_bottom -> P18
- D7 pad 2: P18 -> middle_bottom
- D8 pad 2: P19 -> middle_home
- D9 pad 1: middle_top -> P20
- D9 pad 2: P20 -> middle_top
Other:
- net class Default removed
