File: output/pcbs/main.kicad_pcb (KiCad board)
At the start: 2 copper layers, 251.9 x 126.1 mm, 114 parts

Commit message: Mounting holes: Added
Parts:
- added D37: , ComboDiode, F.Cu at (109.3, 37.2)
- added HOLE1: , MountingHole_2.2mm_M2_Pad_Via, F.Cu at (81.6, -17.7)
- added HOLE2: , MountingHole_2.2mm_M2_Pad_Via, F.Cu at (137.0, -17.7)
- added HOLE3: , MountingHole_2.2mm_M2_Pad_Via, F.Cu at (21.3, -23.2)
- added HOLE4: , MountingHole_2.2mm_M2_Pad_Via, F.Cu at (197.3, -23.2)
- added HOLE5: , MountingHole_2.2mm_M2_Pad_Via, F.Cu at (82.8, 24.8)
- added HOLE6: , MountingHole_2.2mm_M2_Pad_Via, F.Cu at (135.8, 24.8)
- moved D33 168.1 mm to (118.6, -15.1)
- moved S67 168.1 mm to (148.5, 29.4)
- moved S68 168.1 mm to (148.5, 29.4)
- moved S31 168.1 mm to (70.1, 29.4)
- moved S32 168.1 mm to (70.1, 29.4)
- moved S33 168.1 mm to (87.4, 37.4)
- moved S34 168.1 mm to (87.4, 37.4)
- moved S69 168.1 mm to (131.2, 37.4)
- moved S70 168.1 mm to (131.2, 37.4)
- moved S27 168.1 mm to (86.2, -5.04)
- moved S28 168.1 mm to (86.2, -5.04)
- moved D15 168.1 mm to (100.0, -15.1)
- moved S19 168.1 mm to (61.0, 4.15)
- moved S20 168.1 mm to (61.0, 4.15)
- moved S25 168.1 mm to (78.2, 12.2)
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Connections:
- D1 pad 1: P18 -> pinky_bottom
- D10 pad 1: P18 -> index_bottom
- D11 pad 2: index_home -> P19
- D12 pad 1: P20 -> index_top
- D12 pad 2: index_top -> P20
- D13 pad 2: inner_bottom -> P18
- D14 pad 2: inner_home -> P19
- D15 pad 1: P20 -> inner_top
- D15 pad 2: inner_top -> P20
- D17 pad 1: P19 -> home_thumb
- D17 pad 2: home_thumb -> P19
- D18 pad 1: P18 -> far_thumb
- D19 pad 2: mirror_pinky_bottom -> P4
- D2 pad 2: pinky_home -> P19
- D20 pad 1: P5 -> mirror_pinky_home
- D20 pad 2: mirror_pinky_home -> P5
- D21 pad 1: P6 -> mirror_pinky_top
- D21 pad 2: mirror_pinky_top -> P6
- D22 pad 1: P4 -> mirror_ring_bottom
- D24 pad 1: P6 -> mirror_ring_top
- D24 pad 2: mirror_ring_top -> P6
- D25 pad 1: P4 -> mirror_middle_bottom
- D25 pad 2: mirror_middle_bottom -> P4
- D27 pad 1: P6 -> mirror_middle_top
- D28 pad 1: P4 -> mirror_index_bottom
- D29 pad 1: P5 -> mirror_index_home
- D29 pad 2: mirror_index_home -> P5
- D3 pad 1: P20 -> pinky_top
- D3 pad 2: pinky_top -> P20
- D30 pad 2: mirror_index_top -> P6
- D31 pad 1: P4 -> mirror_inner_bottom
- D32 pad 1: P5 -> mirror_inner_home
- D32 pad 2: mirror_inner_home -> P5
- D33 pad 2: mirror_inner_top -> P6
- D34 pad 2: mirror_near_thumb -> P6
- D35 pad 1: P5 -> mirror_home_thumb
- D35 pad 2: mirror_home_thumb -> P5
- D36 pad 1: P4 -> mirror_far_thumb
- D36 pad 2: mirror_far_thumb -> P4
- D4 pad 1: P18 -> ring_bottom
- D5 pad 1: P19 -> ring_home
- D5 pad 2: ring_home -> P19
- D7 pad 1: P18 -> middle_bottom
- D7 pad 2: middle_bottom -> P18
- D8 pad 2: middle_home -> P19
- D9 pad 1: P20 -> middle_top
- D9 pad 2: middle_top -> P20
- JST1 pad 2: GND -> slider_positive
- ROT1 pad 1: GND -> rotary_diode
- ROT1 pad 2: GND -> P14
- T1 pad 1: GND -> slider_positive
Other:
- net class Default added: clearance 0.2, trace_width 0.25, via_dia 0.8, via_drill 0.4
