File: output/pcbs/balbuzard.kicad_pcb (KiCad board)
At the start: 2 copper layers, 251.9 x 126.1 mm, 121 parts

Commit message: Fix issue with thumb mirror not reversing switch pins
Connections:
- S67 pad 1: mirror_near_thumb -> P14
- S67 pad 2: P14 -> mirror_near_thumb
- S68 pad 1: mirror_near_thumb -> P14
- S68 pad 2: P14 -> mirror_near_thumb
- S69 pad 1: mirror_home_thumb -> P14
- S69 pad 2: P14 -> mirror_home_thumb
- S70 pad 1: mirror_home_thumb -> P14
- S70 pad 2: P14 -> mirror_home_thumb
- S71 pad 1: mirror_far_thumb -> P14
- S71 pad 2: P14 -> mirror_far_thumb
- S72 pad 1: mirror_far_thumb -> P14
- S72 pad 2: P14 -> mirror_far_thumb
Changed lines of the file:
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@@
       (pad "" np_thru_hole circle (at 5.08 0) (size 1.7018 1.7018) (drill 1.7018) (layers *.Cu *.Mask))
       (pad "" np_thru_hole circle (at -5.08 0) (size 1.7018 1.7018) (drill 1.7018) (layers *.Cu *.Mask))
-            (pad 1 thru_hole circle (at 2.54 -5.08) (size 2.286 2.286) (drill 1.4986) (layers *.Cu *.Mask) (net 46 "mirror_near_thumb"))
-            (pad 2 thru_hole circle (at -3.81 -2.54) (size 2.286 2.286) (drill 1.4986) (layers *.Cu *.Mask) (net 25 "P14"))
+            (pad 1 thru_hole circle (at 2.54 -5.08) (size 2.286 2.286) (drill 1.4986) (layers *.Cu *.Mask) (net 25 "P14"))
+            (pad 2 thru_hole circle (at -3.81 -2.54) (size 2.286 2.286) (drill 1.4986) (layers *.Cu *.Mask) (net 46 "mirror_near_thumb"))
           )
       (module PG1350 (layer F.Cu)
@@
       (pad "" np_thru_hole circle (at 5.5 0) (size 1.7018 1.7018) (drill 1.7018) (layers *.Cu *.Mask))
       (pad "" np_thru_hole circle (at -5.5 0) (size 1.7018 1.7018) (drill 1.7018) (layers *.Cu *.Mask))
-            (pad 1 thru_hole circle (at 5 -3.8) (size 2.032 2.032) (drill 1.27) (layers *.Cu *.Mask) (net 46 "mirror_near_thumb"))
-            (pad 2 thru_hole circle (at 0 -5.9) (size 2.032 2.032) (drill 1.27) (layers *.Cu *.Mask) (net 25 "P14"))
+            (pad 1 thru_hole circle (at 5 -3.8) (size 2.032 2.032) (drill 1.27) (layers *.Cu *.Mask) (net 25 "P14"))
+            (pad 2 thru_hole circle (at 0 -5.9) (size 2.032 2.032) (drill 1.27) (layers *.Cu *.Mask) (net 46 "mirror_near_thumb"))
           )
     (module ComboDiode (layer F.Cu)
@@
       (pad "" np_thru_hole circle (at 5.08 0) (size 1.7018 1.7018) (drill 1.7018) (layers *.Cu *.Mask))
       (pad "" np_thru_hole circle (at -5.08 0) (size 1.7018 1.7018) (drill 1.7018) (layers *.Cu *.Mask))
-            (pad 1 thru_hole circle (at 2.54 -5.08) (size 2.286 2.286) (drill 1.4986) (layers *.Cu *.Mask) (net 47 "mirror_home_thumb"))
-            (pad 2 thru_hole circle (at -3.81 -2.54) (size 2.286 2.286) (drill 1.4986) (layers *.Cu *.Mask) (net 25 "P14"))
+            (pad 1 thru_hole circle (at 2.54 -5.08) (size 2.286 2.286) (drill 1.4986) (layers *.Cu *.Mask) (net 25 "P14"))
+            (pad 2 thru_hole circle (at -3.81 -2.54) (size 2.286 2.286) (drill 1.4986) (layers *.Cu *.Mask) (net 47 "mirror_home_thumb"))
           )
       (module PG1350 (layer F.Cu)
@@
       (pad "" np_thru_hole circle (at 5.5 0) (size 1.7018 1.7018) (drill 1.7018) (layers *.Cu *.Mask))
       (pad "" np_thru_hole circle (at -5.5 0) (size 1.7018 1.7018) (drill 1.7018) (layers *.Cu *.Mask))
-            (pad 1 thru_hole circle (at 5 -3.8) (size 2.032 2.032) (drill 1.27) (layers *.Cu *.Mask) (net 47 "mirror_home_thumb"))
-            (pad 2 thru_hole circle (at 0 -5.9) (size 2.032 2.032) (drill 1.27) (layers *.Cu *.Mask) (net 25 "P14"))
+            (pad 1 thru_hole circle (at 5 -3.8) (size 2.032 2.032) (drill 1.27) (layers *.Cu *.Mask) (net 25 "P14"))
+            (pad 2 thru_hole circle (at 0 -5.9) (size 2.032 2.032) (drill 1.27) (layers *.Cu *.Mask) (net 47 "mirror_home_thumb"))
           )
     (module ComboDiode (layer F.Cu)
@@
       (pad "" np_thru_hole circle (at 5.08 0) (size 1.7018 1.7018) (drill 1.7018) (layers *.Cu *.Mask))
       (pad "" np_thru_hole circle (at -5.08 0) (size 1.7018 1.7018) (drill 1.7018) (layers *.Cu *.Mask))
-            (pad 1 thru_hole circle (at 2.54 -5.08) (size 2.286 2.286) (drill 1.4986) (layers *.Cu *.Mask) (net 48 "mirror_far_thumb"))
-            (pad 2 thru_hole circle (at -3.81 -2.54) (size 2.286 2.286) (drill 1.4986) (layers *.Cu *.Mask) (net 25 "P14"))
+            (pad 1 thru_hole circle (at 2.54 -5.08) (size 2.286 2.286) (drill 1.4986) (layers *.Cu *.Mask) (net 25 "P14"))
+            (pad 2 thru_hole circle (at -3.81 -2.54) (size 2.286 2.286) (drill 1.4986) (layers *.Cu *.Mask) (net 48 "mirror_far_thumb"))
           )
       (module PG1350 (layer F.Cu)
@@
       (pad "" np_thru_hole circle (at 5.5 0) (size 1.7018 1.7018) (drill 1.7018) (layers *.Cu *.Mask))
       (pad "" np_thru_hole circle (at -5.5 0) (size 1.7018 1.7018) (drill 1.7018) (layers *.Cu *.Mask))
-            (pad 1 thru_hole circle (at 5 -3.8) (size 2.032 2.032) (drill 1.27) (layers *.Cu *.Mask) (net 48 "mirror_far_thumb"))
-            (pad 2 thru_hole circle (at 0 -5.9) (size 2.032 2.032) (drill 1.27) (layers *.Cu *.Mask) (net 25 "P14"))
+            (pad 1 thru_hole circle (at 5 -3.8) (size 2.032 2.032) (drill 1.27) (layers *.Cu *.Mask) (net 25 "P14"))
+            (pad 2 thru_hole circle (at 0 -5.9) (size 2.032 2.032) (drill 1.27) (layers *.Cu *.Mask) (net 48 "mirror_far_thumb"))
           )
     (module ComboDiode (layer F.Cu)

Commit message: Went ahead and used an autorouter to do traces.  Did 90% of the work for me (hopefully)
Parts:
- moved D15 90.2 mm to (130.6, 69.7)
- moved D33 90.2 mm to (149.2, 69.7)
- moved S39 90.2 mm to (241.2, 67.6)
- moved S40 90.2 mm to (241.2, 67.6)
- moved D26 90.2 mm to (188.7, 64.5)
- moved S67 90.2 mm to (179.0, 114.2)
- moved S68 90.2 mm to (179.0, 114.2)
- moved D7 90.2 mm to (84.7, 78.1)
- moved S55 90.2 mm to (188.2, 89.0)
- moved S56 90.2 mm to (188.2, 89.0)
- moved S7 90.2 mm to (57.1, 72.9)
- moved S8 90.2 mm to (57.1, 72.9)
- moved S63 90.2 mm to (163.0, 79.8)
- moved S64 90.2 mm to (163.0, 79.8)
- moved D36 90.2 mm to (153.7, 137.9)
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Connections:
- D1 pad 1: pinky_bottom -> P18
- D1 pad 2: P18 -> pinky_bottom
- D10 pad 2: P18 -> index_bottom
- D11 pad 1: index_home -> P19
- D13 pad 1: inner_bottom -> P18
- D13 pad 2: P18 -> inner_bottom
- D14 pad 1: inner_home -> P19
- D14 pad 2: P19 -> inner_home
- D15 pad 1: inner_top -> P20
- D15 pad 2: P20 -> inner_top
- D16 pad 2: P20 -> near_thumb
- D17 pad 2: P19 -> home_thumb
- D18 pad 1: far_thumb -> P18
- D18 pad 2: P18 -> far_thumb
- D19 pad 2: P4 -> mirror_pinky_bottom
- D2 pad 1: pinky_home -> P19
- D20 pad 2: P5 -> mirror_pinky_home
- D21 pad 1: mirror_pinky_top -> P6
- D22 pad 2: P4 -> mirror_ring_bottom
- D23 pad 1: mirror_ring_home -> P5
- D23 pad 2: P5 -> mirror_ring_home
- D24 pad 1: mirror_ring_top -> P6
- D25 pad 1: mirror_middle_bottom -> P4
- D26 pad 1: mirror_middle_home -> P5
- D26 pad 2: P5 -> mirror_middle_home
- D27 pad 2: P6 -> mirror_middle_top
- D28 pad 2: P4 -> mirror_index_bottom
- D29 pad 1: mirror_index_home -> P5
- D29 pad 2: P5 -> mirror_index_home
- D3 pad 1: pinky_top -> P20
- D31 pad 1: mirror_inner_bottom -> P4
- D31 pad 2: P4 -> mirror_inner_bottom
- D32 pad 1: mirror_inner_home -> P5
- D32 pad 2: P5 -> mirror_inner_home
- D33 pad 1: mirror_inner_top -> P6
- D35 pad 1: mirror_home_thumb -> P5
- D35 pad 2: P5 -> mirror_home_thumb
- D36 pad 1: mirror_far_thumb -> P4
- D37 pad 1: rotary_diode -> P15
- D37 pad 2: P15 -> rotary_diode
- D5 pad 1: ring_home -> P19
- D5 pad 2: P19 -> ring_home
- D6 pad 1: ring_top -> P20
- D7 pad 2: P18 -> middle_bottom
- D9 pad 1: middle_top -> P20
Routing:
- net P9: track 0.00 -> 344.1 mm, vias 0 -> 1
- net P10: track 0.00 -> 299.5 mm, vias 0 -> 1
- net P8: track 0.00 -> 269.8 mm
- net P16: track 0.00 -> 224.0 mm, vias 0 -> 2
- net P4: track 0.00 -> 194.0 mm, vias 0 -> 6
- net P18: track 0.00 -> 185.4 mm, vias 0 -> 6
- net P20: track 0.00 -> 183.2 mm, vias 0 -> 9
- net P5: track 0.00 -> 182.3 mm, vias 0 -> 6
- net P7: track 0.00 -> 179.1 mm, vias 0 -> 1
- net P6: track 0.00 -> 178.7 mm, vias 0 -> 7
- net P14: track 0.00 -> 175.4 mm
- net P19: track 0.00 -> 170.8 mm, vias 0 -> 7
- net GND: track 0.00 -> 93.7 mm
- net P0: track 0.00 -> 65.5 mm, vias 0 -> 1
- net P21: track 0.00 -> 37.3 mm
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Other:
- net class Default removed
