File: rev1/balbuzard.kicad_pcb (KiCad board)
At the start: 2 copper layers, 251.9 x 126.1 mm, 121 parts

Commit message: Routed individual keys, added info on progress
Parts:
- moved S10 97.4 mm to (65.3, 63.3)
- moved S9 97.4 mm to (65.3, 63.3)
- moved OLED1 97.4 mm to (134.4, 125.1)
- moved D18 97.4 mm to (126.3, 145.5), turned to -25 degrees
- moved S7 97.4 mm to (57.3, 80.5)
- moved S8 97.4 mm to (57.3, 80.5)
- moved S71 97.4 mm to (157.4, 153.0)
- moved S72 97.4 mm to (157.4, 153.0)
- moved S11 97.4 mm to (73.4, 46.1)
- moved S12 97.4 mm to (73.4, 46.1)
- moved D15 97.4 mm to (130.8, 77.3)
- moved S5 97.4 mm to (46.9, 58.0)
- moved S6 97.4 mm to (46.9, 58.0)
- moved D36 97.4 mm to (153.9, 145.5)
- moved S41 97.4 mm to (233.3, 58.0)
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Connections:
- D1 pad 1: pinky_bottom -> P18
- D10 pad 1: index_bottom -> P18
- D10 pad 2: P18 -> index_bottom
- D12 pad 1: index_top -> P20
- D12 pad 2: P20 -> index_top
- D13 pad 1: inner_bottom -> P18
- D13 pad 2: P18 -> inner_bottom
- D15 pad 1: inner_top -> P20
- D16 pad 1: near_thumb -> P20
- D16 pad 2: P20 -> near_thumb
- D17 pad 1: home_thumb -> P19
- D17 pad 2: P19 -> home_thumb
- D18 pad 2: P18 -> far_thumb
- D19 pad 2: P4 -> mirror_pinky_bottom
- D2 pad 1: pinky_home -> P19
- D2 pad 2: P19 -> pinky_home
- D22 pad 2: P4 -> mirror_ring_bottom
- D23 pad 2: P5 -> mirror_ring_home
- D24 pad 2: P6 -> mirror_ring_top
- D26 pad 1: mirror_middle_home -> P5
- D27 pad 1: mirror_middle_top -> P6
- D27 pad 2: P6 -> mirror_middle_top
- D28 pad 1: mirror_index_bottom -> P4
- D28 pad 2: P4 -> mirror_index_bottom
- D29 pad 1: mirror_index_home -> P5
- D29 pad 2: P5 -> mirror_index_home
- D3 pad 1: pinky_top -> P20
- D30 pad 2: P6 -> mirror_index_top
- D31 pad 1: mirror_inner_bottom -> P4
- D31 pad 2: P4 -> mirror_inner_bottom
- D32 pad 1: mirror_inner_home -> P5
- D32 pad 2: P5 -> mirror_inner_home
- D33 pad 2: P6 -> mirror_inner_top
- D34 pad 1: mirror_near_thumb -> P6
- D35 pad 1: mirror_home_thumb -> P5
- D36 pad 1: mirror_far_thumb -> P4
- D36 pad 2: P4 -> mirror_far_thumb
- D37 pad 2: P15 -> rotary_diode
- D4 pad 2: P18 -> ring_bottom
- D5 pad 2: P19 -> ring_home
- D6 pad 1: ring_top -> P20
- D7 pad 1: middle_bottom -> P18
- D7 pad 2: P18 -> middle_bottom
- D8 pad 1: middle_home -> P19
- D9 pad 1: middle_top -> P20
- D9 pad 2: P20 -> middle_top
Routing:
- net P10: track 0.00 -> 24.3 mm
- net P9: track 0.00 -> 24.3 mm
- net P8: track 0.00 -> 24.3 mm
- net P14: track 0.00 -> 24.3 mm
- net P16: track 0.00 -> 24.3 mm
- net P7: track 0.00 -> 24.3 mm
- net middle_top: track 0.00 -> 17.3 mm
- net mirror_ring_bottom: track 0.00 -> 17.0 mm
- net mirror_middle_top: track 0.00 -> 14.8 mm
- net mirror_ring_home: track 0.00 -> 13.1 mm
- net P19: track 0.00 -> 13.0 mm
- net P5: track 0.00 -> 13.0 mm
- net P4: track 0.00 -> 13.0 mm
- net P18: track 0.00 -> 13.0 mm
- net P20: track 0.00 -> 13.0 mm
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Other:
- net class Default removed

Commit message: Removed routing, found a better way
Parts:
- moved S10 97.4 mm to (34.5, -29.1)
- moved S9 97.4 mm to (34.5, -29.1)
- moved OLED1 97.4 mm to (103.6, 32.7)
- moved D18 97.4 mm to (95.5, 53.1), turned to 155 degrees
- moved S7 97.4 mm to (26.5, -11.9)
- moved S8 97.4 mm to (26.5, -11.9)
- moved S71 97.4 mm to (126.6, 60.6)
- moved S72 97.4 mm to (126.6, 60.6)
- moved S11 97.4 mm to (42.6, -46.3)
- moved S12 97.4 mm to (42.6, -46.3)
- moved D15 97.4 mm to (100.0, -15.1)
- moved S5 97.4 mm to (16.1, -34.4)
- moved S6 97.4 mm to (16.1, -34.4)
- moved D36 97.4 mm to (123.1, 53.1)
- moved S41 97.4 mm to (202.6, -34.4)
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Connections:
- D1 pad 1: P18 -> pinky_bottom
- D10 pad 1: P18 -> index_bottom
- D10 pad 2: index_bottom -> P18
- D12 pad 1: P20 -> index_top
- D12 pad 2: index_top -> P20
- D13 pad 1: P18 -> inner_bottom
- D13 pad 2: inner_bottom -> P18
- D15 pad 1: P20 -> inner_top
- D16 pad 1: P20 -> near_thumb
- D16 pad 2: near_thumb -> P20
- D17 pad 1: P19 -> home_thumb
- D17 pad 2: home_thumb -> P19
- D18 pad 2: far_thumb -> P18
- D19 pad 2: mirror_pinky_bottom -> P4
- D2 pad 1: P19 -> pinky_home
- D2 pad 2: pinky_home -> P19
- D22 pad 2: mirror_ring_bottom -> P4
- D23 pad 2: mirror_ring_home -> P5
- D24 pad 2: mirror_ring_top -> P6
- D26 pad 1: P5 -> mirror_middle_home
- D27 pad 1: P6 -> mirror_middle_top
- D27 pad 2: mirror_middle_top -> P6
- D28 pad 1: P4 -> mirror_index_bottom
- D28 pad 2: mirror_index_bottom -> P4
- D29 pad 1: P5 -> mirror_index_home
- D29 pad 2: mirror_index_home -> P5
- D3 pad 1: P20 -> pinky_top
- D30 pad 2: mirror_index_top -> P6
- D31 pad 1: P4 -> mirror_inner_bottom
- D31 pad 2: mirror_inner_bottom -> P4
- D32 pad 1: P5 -> mirror_inner_home
- D32 pad 2: mirror_inner_home -> P5
- D33 pad 2: mirror_inner_top -> P6
- D34 pad 1: P6 -> mirror_near_thumb
- D35 pad 1: P5 -> mirror_home_thumb
- D36 pad 1: P4 -> mirror_far_thumb
- D36 pad 2: mirror_far_thumb -> P4
- D37 pad 2: rotary_diode -> P15
- D4 pad 2: ring_bottom -> P18
- D5 pad 2: ring_home -> P19
- D6 pad 1: P20 -> ring_top
- D7 pad 1: P18 -> middle_bottom
- D7 pad 2: middle_bottom -> P18
- D8 pad 1: P19 -> middle_home
- D9 pad 1: P20 -> middle_top
- D9 pad 2: middle_top -> P20
Routing:
- net P10: track 24.3 -> 0.00 mm
- net P9: track 24.3 -> 0.00 mm
- net P8: track 24.3 -> 0.00 mm
- net P14: track 24.3 -> 0.00 mm
- net P16: track 24.3 -> 0.00 mm
- net P7: track 24.3 -> 0.00 mm
- net middle_top: track 17.3 -> 0.00 mm
- net mirror_ring_bottom: track 17.0 -> 0.00 mm
- net mirror_middle_top: track 14.8 -> 0.00 mm
- net mirror_ring_home: track 13.1 -> 0.00 mm
- net P19: track 13.0 -> 0.00 mm
- net P5: track 13.0 -> 0.00 mm
- net P4: track 13.0 -> 0.00 mm
- net P18: track 13.0 -> 0.00 mm
- net P20: track 13.0 -> 0.00 mm
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Other:
- net class Default added: clearance 0.2, trace_width 0.25, via_dia 0.8, via_drill 0.4

Commit message: Redid the key / diode tracks to be as straight as possible.
Parts:
- moved S13 175.9 mm to (154.2, 129.1)
- moved S14 175.9 mm to (154.2, 129.1)
- moved S37 175.9 mm to (333.2, 109.5)
- moved S38 175.9 mm to (333.2, 109.5)
- moved D26 175.9 mm to (265.6, 118.9)
- moved D1 175.9 mm to (107.9, 113.0)
- moved S35 175.9 mm to (199.5, 199.8)
- moved S36 175.9 mm to (199.5, 199.8)
- moved S71 175.9 mm to (234.1, 199.8)
- moved S72 175.9 mm to (234.1, 199.8)
- moved D7 175.9 mm to (161.7, 132.5)
- moved S49 175.9 mm to (279.4, 129.1)
- moved S50 175.9 mm to (279.4, 129.1)
- moved D21 175.9 mm to (302.6, 108.3)
- moved D3 175.9 mm to (131.0, 108.3)
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Connections:
- D1 pad 1: pinky_bottom -> P18
- D1 pad 2: P18 -> pinky_bottom
- D10 pad 1: index_bottom -> P18
- D10 pad 2: P18 -> index_bottom
- D11 pad 1: index_home -> P19
- D11 pad 2: P19 -> index_home
- D12 pad 1: index_top -> P20
- D12 pad 2: P20 -> index_top
- D13 pad 2: P18 -> inner_bottom
- D14 pad 1: inner_home -> P19
- D14 pad 2: P19 -> inner_home
- D15 pad 1: inner_top -> P20
- D16 pad 1: near_thumb -> P20
- D16 pad 2: P20 -> near_thumb
- D17 pad 2: P19 -> home_thumb
- D18 pad 1: far_thumb -> P18
- D19 pad 1: mirror_pinky_bottom -> P4
- D2 pad 1: pinky_home -> P19
- D20 pad 1: mirror_pinky_home -> P5
- D20 pad 2: P5 -> mirror_pinky_home
- D21 pad 1: mirror_pinky_top -> P6
- D21 pad 2: P6 -> mirror_pinky_top
- D23 pad 1: mirror_ring_home -> P5
- D23 pad 2: P5 -> mirror_ring_home
- D24 pad 1: mirror_ring_top -> P6
- D25 pad 1: mirror_middle_bottom -> P4
- D25 pad 2: P4 -> mirror_middle_bottom
- D26 pad 1: mirror_middle_home -> P5
- D26 pad 2: P5 -> mirror_middle_home
- D27 pad 1: mirror_middle_top -> P6
- D28 pad 1: mirror_index_bottom -> P4
- D28 pad 2: P4 -> mirror_index_bottom
- D29 pad 1: mirror_index_home -> P5
- D29 pad 2: P5 -> mirror_index_home
- D30 pad 1: mirror_index_top -> P6
- D30 pad 2: P6 -> mirror_index_top
- D31 pad 2: P4 -> mirror_inner_bottom
- D32 pad 1: mirror_inner_home -> P5
- D32 pad 2: P5 -> mirror_inner_home
- D33 pad 1: mirror_inner_top -> P6
- D34 pad 2: P6 -> mirror_near_thumb
- D35 pad 2: P5 -> mirror_home_thumb
- D36 pad 1: mirror_far_thumb -> P4
- D36 pad 2: P4 -> mirror_far_thumb
- D37 pad 1: rotary_diode -> P15
- D37 pad 2: P15 -> rotary_diode
- D5 pad 1: ring_home -> P19
- D5 pad 2: P19 -> ring_home
- D6 pad 1: ring_top -> P20
- D7 pad 1: middle_bottom -> P18
- D8 pad 1: middle_home -> P19
- D9 pad 1: middle_top -> P20
Routing:
- net P14: track 0.00 -> 23.6 mm
- net P7: track 0.00 -> 23.6 mm
- net P10: track 0.00 -> 23.6 mm
- net P16: track 0.00 -> 23.6 mm
- net P8: track 0.00 -> 23.6 mm
- net P9: track 0.00 -> 23.6 mm
- net middle_top: track 0.00 -> 16.8 mm
- net mirror_middle_top: track 0.00 -> 16.6 mm
- net mirror_ring_bottom: track 0.00 -> 14.8 mm
- net P18: track 0.00 -> 13.0 mm
- net P20: track 0.00 -> 13.0 mm
- net P19: track 0.00 -> 13.0 mm
- net P4: track 0.00 -> 13.0 mm
- net P6: track 0.00 -> 13.0 mm
- net mirror_ring_home: track 0.00 -> 12.7 mm
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Other:
- net class Default removed

Commit message: Went ahead and used an autorouter to do traces.  Did 90% of the work for me (hopefully)
Parts:
- moved HOLE4 94.2 mm to (227.9, 61.7)
- moved D2 94.2 mm to (47.3, 68.4)
- moved HOLE5 94.2 mm to (113.3, 109.7)
- moved S51 94.2 mm to (194.5, 57.4)
- moved S52 94.2 mm to (194.5, 57.4)
- moved D9 94.2 mm to (97.8, 50.0)
- moved D11 94.2 mm to (107.0, 75.3)
- moved D13 94.2 mm to (116.2, 100.5)
- moved D17 94.2 mm to (125.4, 125.8)
- moved D3 94.2 mm to (54.1, 53.9)
- moved S65 94.2 mm to (154.9, 62.6)
- moved S66 94.2 mm to (154.9, 62.6)
- moved S45 94.2 mm to (214.6, 55.7)
- moved S46 94.2 mm to (214.6, 55.7)
- moved S57 94.2 mm to (180.2, 71.8)
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Connections:
- D10 pad 1: P18 -> index_bottom
- D11 pad 2: index_home -> P19
- D12 pad 1: P20 -> index_top
- D12 pad 2: index_top -> P20
- D13 pad 1: inner_bottom -> P18
- D15 pad 2: P20 -> inner_top
- D16 pad 1: P20 -> near_thumb
- D18 pad 2: P18 -> far_thumb
- D19 pad 1: P4 -> mirror_pinky_bottom
- D19 pad 2: P4 -> mirror_pinky_bottom
- D20 pad 1: P5 -> mirror_pinky_home
- D21 pad 2: mirror_pinky_top -> P6
- D22 pad 2: P4 -> mirror_ring_bottom
- D25 pad 2: mirror_middle_bottom -> P4
- D27 pad 1: P6 -> mirror_middle_top
- D27 pad 2: P6 -> mirror_middle_top
- D28 pad 1: P4 -> mirror_index_bottom
- D3 pad 1: pinky_top -> P20
- D30 pad 1: P6 -> mirror_index_top
- D30 pad 2: mirror_index_top -> P6
- D31 pad 1: mirror_inner_bottom -> P4
- D34 pad 2: mirror_near_thumb -> P6
- D35 pad 1: mirror_home_thumb -> P5
- D36 pad 2: mirror_far_thumb -> P4
- D7 pad 1: P18 -> middle_bottom
- D7 pad 2: P18 -> middle_bottom
- D8 pad 1: P19 -> middle_home
Routing:
- net P9: track 23.6 -> 344.1 mm, vias 0 -> 1
- net P10: track 23.6 -> 299.5 mm, vias 0 -> 1
- net P8: track 23.6 -> 269.8 mm
- net P16: track 23.6 -> 224.0 mm, vias 0 -> 2
- net P4: track 13.0 -> 194.0 mm, vias 0 -> 6
- net P18: track 13.0 -> 185.4 mm, vias 0 -> 6
- net P5: track 10.8 -> 182.3 mm, vias 0 -> 6
- net P20: track 13.0 -> 183.2 mm, vias 0 -> 9
- net P6: track 13.0 -> 178.7 mm, vias 0 -> 7
- net P19: track 13.0 -> 170.8 mm, vias 0 -> 7
- net P7: track 23.6 -> 179.1 mm, vias 0 -> 1
- net P14: track 23.6 -> 175.4 mm
- net GND: track 0.00 -> 93.7 mm
- net P0: track 0.00 -> 65.5 mm, vias 0 -> 1
- net P21: track 0.00 -> 37.3 mm
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